Commit message: mesa en urdf

File: ros_ur_driver/install/ur_description/share/ur_description/urdf/ur_macro.xacro (robot description, xacro)
@@ -227,4 +227,27 @@
       </xacro:cylinder_inertial>
     </link>
+    <!--||||||||||||||||||||||||||||||||||||||||||||||||||||||||||||||||||||||||||||||||||||||||||||||||||||||||||||||||||||||||||||||||||||-->
+    <link name="mesa">
+      <visual>
+        <!--<origin xyz="0.76884 -0.27794 -0.16726" rpy="-0.0054 -0.0053 0.0116"/>-->
+        <origin xyz="0 0 0" rpy="0 0 0"/>
+        <geometry>
+          <mesh filename="file://$(find ur_description)/meshes/ur10/visual/03_Estación.stl" scale="0.001 0.001 0.001"/>
+        </geometry>
+        <material name="${wrist_3_visual_material_name}">
+          <color rgba="${wrist_3_visual_material_color}"/>
+        </material>
+      </visual>
+      <collision>
+        <origin xyz="0 0 0" rpy="0 0 0"/>
+        <geometry>
+          <mesh filename="file://$(find ur_description)/meshes/ur10/collision/03_Estación.stl" scale="0.001 0.001 0.001"/>
+        </geometry>
+      </collision>
+      <!--<xacro:cylinder_inertial radius="${wrist_3_inertia_radius}" length="${wrist_3_inertia_length}"  mass="${wrist_3_mass}">
+        <origin xyz="0.0 0.0 ${-0.5 * wrist_3_inertia_length}" rpy="0 0 0" />
+      </xacro:cylinder_inertial>-->
+    </link>
+    <!--||||||||||||||||||||||||||||||||||||||||||||||||||||||||||||||||||||||||||||||||||||||||||||||||||||||||||||||||||||||||||||||||||||-->
     <!-- joints - main serial chain -->
     <joint name="${prefix}base_link-base_link_inertia" type="fixed">
@@ -310,4 +333,13 @@
       <dynamics damping="0" friction="0"/>
     </joint>
+    <!-- ||||||||||||||||||||||||||||||||||||||||||||||||||||||||||||||||||||||||||||||||||||||||||||||||||||||||||||||||||||||||||||||||||| -->
+    <joint name="joint_mesa" type="fixed">
+      <parent link="${prefix}base_link_inertia" />
+      <child link="mesa" />
+      <!--<origin xyz="0.76884 -0.27794 -0.16726" rpy="-0.0054 -0.0053 3.153192654"/>LO QUE DEBERIA SER, PERO ESTA MAL EL MODELO-->
+      <origin xyz="0.74884 -0.27794 -0.17726" rpy="-0.0054 -0.0053 3.153192654"/>
+      <axis xyz="0 0 1" />
+    </joint>
+    <!-- ||||||||||||||||||||||||||||||||||||||||||||||||||||||||||||||||||||||||||||||||||||||||||||||||||||||||||||||||||||||||||||||||||| -->
     <!-- ROS-Industrial 'base' frame - base_link to UR 'Base' Coordinates transform -->
     <link name="${prefix}base"/>
