Commit message: antes de prueba salsa secreta

File: Universal_Robots_ROS2_Description/urdf/ur_macro.xacro (robot description, xacro)
@@ -258,5 +258,5 @@
     <link name="mesa">
       <visual>
-        <origin xyz="0 0 0" rpy="0 0 0"/>
+        <origin xyz="0 0 0" rpy="0 0 ${pi}"/>
         <geometry>
           <mesh filename="file://$(find ur_description)/meshes/ur10/visual/03_Estación.stl" scale="0.001 0.001 0.001"/>
@@ -286,5 +286,5 @@
            link/frame) to introduce the necessary rotation over Z (of pi rad).
       -->
-      <origin xyz="0 0 0" rpy="0 0 ${pi}" />
+      <origin xyz="0 0 0" rpy="0 0 0" />
     </joint>
     <joint name="${tf_prefix}shoulder_pan_joint" type="revolute">
@@ -362,7 +362,7 @@
     <!-- ||||||||||||||||||||||||||||||||||||||||||||||||||||||||||||||||||||||||||||||||||||||||||||||||||||||||||||||||||||||||||||||||||| -->
     <joint name="joint_mesa" type="fixed">
-      <parent link="${tf_prefix}base_link_inertia" />
+      <parent link="${tf_prefix}base_link" />
       <child link="mesa" />
-      <origin xyz="0.74884 -0.27794 -0.17726" rpy="-0.0054 -0.0053 3.153192654"/>
+      <origin xyz="-0.76884 0.27794 -0.16726" rpy="-0.0054 -0.0053 3.153192654"/>
       <axis xyz="0 0 1" />
     </joint>

Commit message: cambios de posicion de mesa

File: Universal_Robots_ROS2_Description/urdf/ur_macro.xacro (robot description, xacro)
@@ -258,5 +258,5 @@
     <link name="mesa">
       <visual>
-        <origin xyz="0 0 0" rpy="0 0 ${pi}"/>
+        <origin xyz="0 0 0" rpy="0 0 0"/>
         <geometry>
           <mesh filename="file://$(find ur_description)/meshes/ur10/visual/03_Estación.stl" scale="0.001 0.001 0.001"/>
@@ -362,7 +362,7 @@
     <!-- ||||||||||||||||||||||||||||||||||||||||||||||||||||||||||||||||||||||||||||||||||||||||||||||||||||||||||||||||||||||||||||||||||| -->
     <joint name="joint_mesa" type="fixed">
-      <parent link="${tf_prefix}base_link" />
+      <parent link="${tf_prefix}base_link_inertia" />
       <child link="mesa" />
-      <origin xyz="-0.76884 0.27794 -0.16726" rpy="-0.0054 -0.0053 3.153192654"/>
+      <origin xyz="0.74884 -0.27794 -0.17726" rpy="-0.0054 -0.0053 3.153192654"/>
       <axis xyz="0 0 1" />
     </joint>

Commit message: mesa orientada con percha inflada

File: Universal_Robots_ROS2_Description/urdf/ur_macro.xacro (robot description, xacro)
@@ -258,13 +258,13 @@
     <link name="mesa">
       <visual>
-        <origin xyz="0 0 0" rpy="0 0 0"/>
-        <geometry>
-          <mesh filename="file://$(find ur_description)/meshes/ur10/visual/03_Estación.stl" scale="0.001 0.001 0.001"/>
-        </geometry>
-      </visual>
-      <collision>
-        <origin xyz="0 0 0" rpy="0 0 0"/>
-        <geometry>
-          <mesh filename="file://$(find ur_description)/meshes/ur10/collision/03_Estación.stl" scale="0.001 0.001 0.001"/>
+        <origin xyz="0 0 0" rpy="0 0 ${pi}"/>
+        <geometry>
+          <mesh filename="file://$(find ur_description)/meshes/ur10/visual/05_Estación_Gorda.stl" scale="0.001 0.001 0.001"/>
+        </geometry>
+      </visual>
+      <collision>
+        <origin xyz="0 0 0" rpy="0 0 ${pi}"/>
+        <geometry>
+          <mesh filename="file://$(find ur_description)/meshes/ur10/collision/05_Estación_Gorda.stl" scale="0.001 0.001 0.001"/>
         </geometry>
       </collision>
@@ -362,7 +362,7 @@
     <!-- ||||||||||||||||||||||||||||||||||||||||||||||||||||||||||||||||||||||||||||||||||||||||||||||||||||||||||||||||||||||||||||||||||| -->
     <joint name="joint_mesa" type="fixed">
-      <parent link="${tf_prefix}base_link_inertia" />
+      <parent link="${tf_prefix}base_link" />
       <child link="mesa" />
-      <origin xyz="0.74884 -0.27794 -0.17726" rpy="-0.0054 -0.0053 3.153192654"/>
+      <origin xyz="0.76884 -0.27794 -0.16726" rpy="-0.0054 -0.0053 0.0116"/>
       <axis xyz="0 0 1" />
     </joint>
